File: ai03_pcb_guide/Deej keypad/Deej keypad.sch (KiCad schematic (older format))
At the start: 26 parts

Commit message: saving changes
Parts:
- removed D5, D8: D_Small, Diodes_SMD:D_SOD-123, symbol Device:D_Small
- renumbered D12 to D10, D13 to D11, D14 to D12, D6 to D5, D7 to D6, D9 to D7, D10 to D8, D11 to D9
Changed lines of the file:
@@
 $EndComp
-$Comp
-L Device:D_Small D8
-U 1 1 6763414F
-P 5050 3100
-F 0 "D8" V 5096 3032 50  0000 R CNN
-F 1 "D_Small" V 5005 3032 50  0000 R CNN
-F 2 "Diodes_SMD:D_SOD-123" V 5050 3100 50  0001 C CNN
-F 3 "~" V 5050 3100 50  0001 C CNN
-	1    5050 3100
-	0    -1   -1   0
-$EndComp
-Wire Wire Line
-	5050 3000 5050 2900
 $Comp
 L MX_Alps_Hybrid:MX-NoLED MX10
@@
 $EndComp
 $Comp
-L Device:D_Small D12
+L Device:D_Small D10
 U 1 1 676358A6
 P 5550 3100
-F 0 "D12" V 5596 3032 50  0000 R CNN
+F 0 "D10" V 5596 3032 50  0000 R CNN
 F 1 "D_Small" V 5505 3032 50  0000 R CNN
 F 2 "Diodes_SMD:D_SOD-123" V 5550 3100 50  0001 C CNN
@@
 	4050 3850 4050 3750
 $Comp
-L Device:D_Small D5
-U 1 1 6763B094
-P 4550 3100
-F 0 "D5" V 4596 3032 50  0000 R CNN
-F 1 "D_Small" V 4505 3032 50  0000 R CNN
-F 2 "Diodes_SMD:D_SOD-123" V 4550 3100 50  0001 C CNN
-F 3 "~" V 4550 3100 50  0001 C CNN
-	1    4550 3100
-	0    -1   -1   0
-$EndComp
-$Comp
-L Device:D_Small D9
-U 1 1 6763B09E
-P 5050 3100
-F 0 "D9" V 5096 3032 50  0000 R CNN
-F 1 "D_Small" V 5005 3032 50  0000 R CNN
-F 2 "Diodes_SMD:D_SOD-123" V 5050 3100 50  0001 C CNN
-F 3 "~" V 5050 3100 50  0001 C CNN
-	1    5050 3100
-	0    -1   -1   0
-$EndComp
-$Comp
 L MX_Alps_Hybrid:MX-NoLED MX5
 U 1 1 6763B0A8
@@
 $EndComp
 $Comp
-L Device:D_Small D6
+L Device:D_Small D5
 U 1 1 6763B0B2
 P 4550 3950
-F 0 "D6" V 4596 3882 50  0000 R CNN
+F 0 "D5" V 4596 3882 50  0000 R CNN
 F 1 "D_Small" V 4505 3882 50  0000 R CNN
 F 2 "Diodes_SMD:D_SOD-123" V 4550 3950 50  0001 C CNN
@@
 Wire Wire Line
 	4550 3850 4550 3750
-Connection ~ 4550 3000
-Connection ~ 5050 3000
 $Comp
 L MX_Alps_Hybrid:MX-NoLED MX8
@@
 $EndComp
 $Comp
-L Device:D_Small D10
+L Device:D_Small D8
 U 1 1 6763EE9C
 P 5050 3950
-F 0 "D10" V 5096 3882 50  0000 R CNN
+F 0 "D8" V 5096 3882 50  0000 R CNN
 F 1 "D_Small" V 5005 3882 50  0000 R CNN
 F 2 "Diodes_SMD:D_SOD-123" V 5050 3950 50  0001 C CNN
@@
 $EndComp
 $Comp
-L Device:D_Small D13
+L Device:D_Small D11
 U 1 1 6764039E
 P 5550 3950
-F 0 "D13" V 5596 3882 50  0000 R CNN
+F 0 "D11" V 5596 3882 50  0000 R CNN
 F 1 "D_Small" V 5505 3882 50  0000 R CNN
 F 2 "Diodes_SMD:D_SOD-123" V 5550 3950 50  0001 C CNN
@@
 $EndComp
 $Comp
-L Device:D_Small D7
+L Device:D_Small D6
 U 1 1 676525F5
 P 4550 4800
-F 0 "D7" V 4596 4732 50  0000 R CNN
+F 0 "D6" V 4596 4732 50  0000 R CNN
 F 1 "D_Small" V 4505 4732 50  0000 R CNN
 F 2 "Diodes_SMD:D_SOD-123" V 4550 4800 50  0001 C CNN
@@
 $EndComp
 $Comp
-L Device:D_Small D11
+L Device:D_Small D9
 U 1 1 6765260A
 P 5050 4800
-F 0 "D11" V 5096 4732 50  0000 R CNN
+F 0 "D9" V 5096 4732 50  0000 R CNN
 F 1 "D_Small" V 5005 4732 50  0000 R CNN
 F 2 "Diodes_SMD:D_SOD-123" V 5050 4800 50  0001 C CNN
@@
 $EndComp
 $Comp
-L Device:D_Small D14
+L Device:D_Small D12
 U 1 1 6765261F
 P 5550 4800
-F 0 "D14" V 5596 4732 50  0000 R CNN
+F 0 "D12" V 5596 4732 50  0000 R CNN
 F 1 "D_Small" V 5505 4732 50  0000 R CNN
 F 2 "Diodes_SMD:D_SOD-123" V 5550 4800 50  0001 C CNN
@@
 	4050 3200 4550 3200
 Connection ~ 4550 3200
-Wire Wire Line
-	4550 3200 5050 3200
-Connection ~ 5050 3200
-Wire Wire Line
-	5050 3200 5550 3200
 Wire Wire Line
 	4050 4050 4550 4050
@@
 Text GLabel 4250 2300 1    50   Input ~ 0
 COL0
+Connection ~ 5050 3200
+Wire Wire Line
+	5050 3200 5550 3200
+Wire Wire Line
+	4550 3200 5050 3200
+$Comp
+L Device:D_Small D7
+U 1 1 6763B09E
+P 5050 3100
+F 0 "D7" V 5096 3032 50  0000 R CNN
+F 1 "D_Small" V 5005 3032 50  0000 R CNN
+F 2 "Diodes_SMD:D_SOD-123" V 5050 3100 50  0001 C CNN
+F 3 "~" V 5050 3100 50  0001 C CNN
+	1    5050 3100
+	0    -1   -1   0
+$EndComp
+Wire Wire Line
+	5050 3000 5050 2900
 $EndSCHEMATC
